File: schematics/mcu.kicad_sch (KiCad schematic)
At the start: 13 parts, among them U1 STM32F103VBT6, Y1 16Mhz

Commit message: Update V2
Other:
- note added: "Cload = 2 * (CL - Cstray) CL = 10pF Cstray = 5pF"
